Commit message: add to link3

File: um_description/urdf/um.urdf (robot description, URDF)
Before this commit: robot um, 2 links, 1 joints
Links:
- link link1: geometry visual mesh filename=package://um_description/meshes/link1a.STL scale=1 1 1

Commit message: add um_gazebo for simulation

File: um_description/urdf/um.urdf (robot description, URDF)
Before this commit: robot um, 2 links, 1 joints
Links:
- added link bottom_link, mass 500; collision box size=1 1 0.02; visual box size=1 1 0.02
- added link link2, mass 1; collision mesh filename=package://um_description/meshes/link2.STL scale=1 1 1; visual mesh filename=package://um_description/meshes/link2.STL scale=1 1 1
- added link link3, mass 1; collision mesh filename=package://um_description/meshes/link3.STL scale=1 1 1; visual mesh filename=package://um_description/meshes/link3.STL scale=1 1 1
- added link link4, mass 1; collision mesh filename=package://um_description/meshes/link4.STL scale=1 1 1; visual mesh filename=package://um_description/meshes/link4.STL scale=1 1 1
- added link link5, mass 1; collision mesh filename=package://um_description/meshes/link5.STL scale=1 1 1; visual mesh filename=package://um_description/meshes/link5.STL scale=1 1 1
- link base_link: mass None -> 1; geometry collision mesh filename=package://um_description/meshes/base.STL scale=1 1 1; visual mesh filename=package://um_description/meshes/base.STL scale=1 1 1
- link link1: mass None -> 1; geometry collision mesh filename=package://um_description/meshes/link1.STL scale=1 1 1; visual mesh filename=package://um_description/meshes/link1.STL scale=1 1 1
Joints:
- added joint bottom_joint: type fixed, parent base_link, child bottom_link, origin xyz=0 0 0 rpy=0 0 0
- added joint joint2: type revolute, parent link1, child link2, origin xyz=0.055 -0.0075 0.1764 rpy=0 0 0, axis 0 0 1, limit lower=-3.1415926 upper=3.1415926 effort=300 velocity=1.0
- added joint joint3: type revolute, parent link2, child link3, origin xyz=0.0349 0 0.0225 rpy=0 0 0, axis 1 0 0, limit lower=-3.1415926 upper=3.1415926 effort=300 velocity=1.0
- added joint joint4: type revolute, parent link3, child link4, origin xyz=0.2655 0 -0.00025 rpy=0 0 0, axis 0 1 0, limit lower=-1.5707963 upper=1.5707963 effort=300 velocity=1.0
- added joint joint5: type revolute, parent link4, child link5, origin xyz=0.1255 0 0 rpy=0 0 0, axis 0 1 0, limit lower=-1.5707963 upper=1.5707963 effort=300 velocity=1.0
- joint joint1: limit lower=0 upper=0.59 effort=100 velocity=1.0 -> lower=0 upper=0.59 effort=300 velocity=1.0; origin xyz=0 0 0 -> xyz=0 0 0 rpy=0 0 0

File: um_description/urdf/um.urdf.xacro (robot description, xacro)
@@ -1,6 +1,6 @@
 <?xml version="1.0"?>
-<robot name="um" xmlns:xacro="http://www.ros.org/wiki/xacro">
-<!--Define the colors used in the um-->
-    <material name="Gray">
+<robot name="um" xmlns:xacro="http://ros.org/wiki/xacro">
+    <!-- Define the colors used in the um -->
+    <material name="Grey">
         <color rgba="0.75 0.75 0.75 1" />
     </material>
@@ -23,14 +23,21 @@
         <color rgba="0 1 0 1"/>
     </material>
-<!-- Define the constants used in the um -->
+    <!-- Define the macros used in um -->
+    <xacro:macro name="inertia_matrix" params="mass">
+        <inertial>
+            <mass value="${mass}" />
+            <inertia ixx="1.0" ixy="0" ixz="0" iyy="0.5" iyz="0" izz="1.0" />
+        </inertial>
+    </xacro:macro>
+    <!-- Define the constants used in the um -->
     <xacro:property name="M_PI" value="3.1415926" />
     <xacro:property name="DAMPING" value="50" />
     <xacro:property name="FRICTION" value="1" />
-<!-- Joint1 properties -->
-    <xacro:property name="JOINT1_EFFORT" value="100" />
+    <!-- Joint1 properties -->
+    <xacro:property name="JOINT1_EFFORT" value="300" />
     <xacro:property name="JOINT1_LOWER" value="0" />
     <xacro:property name="JOINT1_UPPER" value="0.59" />
     <xacro:property name="JOINT1_VEL" value="1.0" />
-<!-- Joint2 properties -->
+    <!-- Joint2 properties -->
     <xacro:property name="JOINT2_COOR" value="0.055 -0.0075 0.1764" />
     <xacro:property name="JOINT2_EFFORT" value="300" />
@@ -38,5 +45,5 @@
     <xacro:property name="JOINT2_UPPER" value="${M_PI}" />
     <xacro:property name="JOINT2_VEL" value="1.0" />
-<!-- Joint 3 properties -->
+    <!-- Joint 3 properties -->
     <xacro:property name="JOINT3_COOR" value="0.0349 0 0.0225" />
     <xacro:property name="JOINT3_EFFORT" value="300" />
@@ -44,5 +51,5 @@
     <xacro:property name="JOINT3_UPPER" value="${M_PI}" />
     <xacro:property name="JOINT3_VEL" value="1.0" />
-<!-- Joint 4 properties -->
+    <!-- Joint 4 properties -->
     <xacro:property name="JOINT4_COOR" value="0.2655 0 -0.00025" />
     <xacro:property name="JOINT4_EFFORT" value="300" />
@@ -50,5 +57,5 @@
     <xacro:property name="JOINT4_UPPER" value="${M_PI/2}" />
     <xacro:property name="JOINT4_VEL" value="1.0" />
-<!-- Joint 5 properties -->
+    <!-- Joint 5 properties -->
     <xacro:property name="JOINT5_COOR" value="0.1255 0 0" />
     <xacro:property name="JOINT5_EFFORT" value="300" />
@@ -56,23 +63,30 @@
     <xacro:property name="JOINT5_UPPER" value="${M_PI/2}" />
     <xacro:property name="JOINT5_VEL" value="1.0" />
-<!--////////////////  BASE LINK  ///////////////////// -->
+<!-- ////////////////  BASE LINK  ///////////////////// -->
     <link name="base_link">
         <visual>
-            <origin xyz="0 0 0" rpy="${M_PI} 0 0" />
+            <origin xyz="0 0 0" rpy="0 0 0" />
             <geometry>
                 <mesh filename="package://um_description/meshes/base.STL" scale="1 1 1" />
             </geometry>
-            <material name="Gray" />
-        </visual>
+            <material name="Grey" />
+        </visual>
+        <collision>
+            <origin xyz="0 0 0" rpy="0 0 0" />
+            <geometry>
+                <mesh filename="package://um_description/meshes/base.STL" scale="1 1 1" />
+            </geometry>
+        </collision>
+        <xacro:inertia_matrix mass="1" />
     </link>
     <joint name="joint1" type="prismatic">
         <parent link="base_link"/>
         <child link="link1"/>
-        <origin xyz="0 0 0" rpy="${M_PI} 0 0" />
+        <origin xyz="0 0 0" rpy="0 0 0" />
         <axis xyz="1 0 0"/>
         <limit effort="${JOINT1_EFFORT}" lower="${JOINT1_LOWER}" upper="${JOINT1_UPPER}" velocity="${JOINT1_VEL}" />
         <dynamics damping="${DAMPING}" friction="${FRICTION}" />
     </joint>
-<!--/////////////////  LINK 1  //////////////////////// -->
+    <!-- /////////////////  LINK 1  //////////////////////// -->
     <link name="link1">
         <visual>
@@ -83,4 +97,11 @@
             <material name="Orange" />
         </visual>
+        <collision>
+            <origin xyz="${JOINT2_COOR}" rpy="0 0 0"/>
+            <geometry>
+                <mesh filename="package://um_description/meshes/link1.STL" scale="1 1 1"/>
+            </geometry>
+        </collision>
+        <xacro:inertia_matrix mass="1" />
     </link>
     <joint name="joint2" type="revolute">
@@ -92,5 +113,5 @@
         <dynamics damping="${DAMPING}" friction="${FRICTION}" />
     </joint>
-<!--/////////////////  LINK 2  //////////////////////// -->
+    <!-- /////////////////  LINK 2  //////////////////////// -->
     <link name="link2">
         <visual>
@@ -99,6 +120,13 @@
                 <mesh filename="package://um_description/meshes/link2.STL" scale="1 1 1" />
             </geometry>
-            <material name="Gray" />
-        </visual>
+            <material name="Grey" />
+        </visual>
+        <collision>
+            <origin xyz="0 0 0" rpy="0 0 0" />
+            <geometry>
+                <mesh filename="package://um_description/meshes/link2.STL" scale="1 1 1" />
+            </geometry>
+        </collision>
+        <xacro:inertia_matrix mass="1" />
     </link>
     <joint name="joint3" type="revolute">
@@ -110,5 +138,5 @@
         <dynamics damping="${DAMPING}" friction="${FRICTION}" />
     </joint>
-<!--/////////////////  LINK 3  //////////////////////// -->
+    <!-- /////////////////  LINK 3  //////////////////////// -->
     <link name="link3">
         <visual>
@@ -119,4 +147,11 @@
             <material name="Orange" />
         </visual>
+        <collision>
+            <origin xyz="0 0 0" rpy="0 0 0" />
+            <geometry>
+                <mesh filename="package://um_description/meshes/link3.STL" scale="1 1 1" />
+            </geometry>
+        </collision>
+        <xacro:inertia_matrix mass="1" />
     </link>
     <joint name="joint4" type="revolute">
@@ -128,5 +163,5 @@
         <dynamics damping="${DAMPING}" friction="${FRICTION}" />
     </joint>
-<!--/////////////////  LINK 4  //////////////////////// -->
+    <!-- /////////////////  LINK 4  //////////////////////// -->
     <link name="link4">
         <visual>
@@ -135,6 +170,13 @@
                 <mesh filename="package://um_description/meshes/link4.STL" scale="1 1 1" />
             </geometry>
-            <material name="Gray" />
-        </visual>
+            <material name="Grey" />
+        </visual>
+        <collision>
+            <origin xyz="0 0 0" rpy="0 0 0" />
+            <geometry>
+                <mesh filename="package://um_description/meshes/link4.STL" scale="1 1 1" />
+            </geometry>
+        </collision>
+        <xacro:inertia_matrix mass="1" />
     </link>
     <joint name="joint5" type="revolute">
@@ -146,5 +188,5 @@
         <dynamics damping="${DAMPING}" friction="${FRICTION}" />
     </joint>
-<!--/////////////////  LINK 5  //////////////////////// -->
+    <!-- /////////////////  LINK 5  //////////////////////// -->
     <link name="link5">
         <visual>
@@ -155,4 +197,55 @@
             <material name="Orange" />
         </visual>
-    </link>
+        <collision>
+            <origin xyz="0 0 0" rpy="0 0 0" />
+            <geometry>
+                <mesh filename="package://um_description/meshes/link5.STL" scale="1 1 1" />
+            </geometry>
+        </collision>
+        <xacro:inertia_matrix mass="1" />
+    </link>
+    <!-- /////////////////  GAZEBO  //////////////////////// -->
+    <!-- Materials of all links in Gazebo -->
+    <gazebo reference="base_link">
+        <material>Gazebo/Grey</material>
+    </gazebo>
+    <gazebo reference="link1">
+        <material>Gazebo/Orange</material>
+    </gazebo>
+    <gazebo reference="link2">
+        <material>Gazebo/Grey</material>
+    </gazebo>
+    <gazebo reference="link3">
+        <material>Gazebo/Orange</material>
+    </gazebo>
+    <gazebo reference="link4">
+        <material>Gazebo/Grey</material>
+    </gazebo>
+    <gazebo reference="link5">
+        <material>Gazebo/Orange</material>
+    </gazebo>
+    <!-- Transmissions for ROS Control -->
+    <xacro:macro name="transmission_block" params="joint_name">
+        <transmission name="tran1">
+            <type>transmission_interface/SimpleTransmission</type>
+            <joint name="${joint_name}">
+                <hardwareInterface>hardware_interface/PositionJointInterface</hardwareInterface>
+            </joint>
+            <actuator name="motor1">
+                <hardwareInterface>hardware_interface/PositionJointInterface</hardwareInterface>
+                <mechanicalReduction>1</mechanicalReduction>
+            </actuator>
+        </transmission>
+    </xacro:macro>
+    <xacro:transmission_block joint_name="joint1" />
+    <xacro:transmission_block joint_name="joint2" />
+    <xacro:transmission_block joint_name="joint3" />
+    <xacro:transmission_block joint_name="joint4" />
+    <xacro:transmission_block joint_name="joint5" />
+    <!-- ros_control plugin -->
+    <gazebo>
+        <plugin name="gazebo_ros_control" filename="libgazebo_ros_control.so">
+            <robotNamespace>/um</robotNamespace>
+        </plugin>
+    </gazebo>
 </robot>
