Commit message: add all links

File: um_description/urdf/um.urdf.xacro (robot description, xacro)
@@ -5,5 +5,5 @@
         <color rgba="0.75 0.75 0.75 1" />
     </material>
-    <material name="Yellow">
+    <material name="Orange">
         <color rgba="1 0.4 0 1"/>
     </material>
@@ -44,8 +44,20 @@
     <xacro:property name="JOINT3_UPPER" value="${M_PI}" />
     <xacro:property name="JOINT3_VEL" value="1.0" />
+<!-- Joint 4 properties -->
+    <xacro:property name="JOINT4_COOR" value="0.2655 0 -0.00025" />
+    <xacro:property name="JOINT4_EFFORT" value="300" />
+    <xacro:property name="JOINT4_LOWER" value="-${M_PI/2}" />
+    <xacro:property name="JOINT4_UPPER" value="${M_PI/2}" />
+    <xacro:property name="JOINT4_VEL" value="1.0" />
+<!-- Joint 5 properties -->
+    <xacro:property name="JOINT5_COOR" value="0.1255 0 0" />
+    <xacro:property name="JOINT5_EFFORT" value="300" />
+    <xacro:property name="JOINT5_LOWER" value="-${M_PI/2}" />
+    <xacro:property name="JOINT5_UPPER" value="${M_PI/2}" />
+    <xacro:property name="JOINT5_VEL" value="1.0" />
 <!--////////////////  BASE LINK  ///////////////////// -->
     <link name="base_link">
         <visual>
-            <origin xyz="0 0 0" rpy="0 0 0" />
+            <origin xyz="0 0 0" rpy="${M_PI} 0 0" />
             <geometry>
                 <mesh filename="package://um_description/meshes/base.STL" scale="1 1 1" />
@@ -57,5 +69,5 @@
         <parent link="base_link"/>
         <child link="link1"/>
-        <origin xyz="0 0 0"/>
+        <origin xyz="0 0 0" rpy="${M_PI} 0 0" />
         <axis xyz="1 0 0"/>
         <limit effort="${JOINT1_EFFORT}" lower="${JOINT1_LOWER}" upper="${JOINT1_UPPER}" velocity="${JOINT1_VEL}" />
@@ -69,5 +81,5 @@
                 <mesh filename="package://um_description/meshes/link1.STL" scale="1 1 1"/>
             </geometry>
-            <material name="Yellow" />
+            <material name="Orange" />
         </visual>
     </link>
@@ -87,5 +99,5 @@
                 <mesh filename="package://um_description/meshes/link2.STL" scale="1 1 1" />
             </geometry>
-            <material name="Blue" />
+            <material name="Gray" />
         </visual>
     </link>
@@ -105,8 +117,42 @@
                 <mesh filename="package://um_description/meshes/link3.STL" scale="1 1 1" />
             </geometry>
-            <material name="Green" />
+            <material name="Orange" />
         </visual>
     </link>
+    <joint name="joint4" type="revolute">
+        <parent link="link3" />
+        <child link="link4" />
+        <origin xyz="${JOINT4_COOR}" rpy="0 0 0" />
+        <axis xyz="0 1 0" />
+        <limit effort="${JOINT4_EFFORT}" lower="${JOINT4_LOWER}" upper="${JOINT4_UPPER}" velocity="${JOINT4_VEL}" />
+        <dynamics damping="${DAMPING}" friction="${FRICTION}" />
+    </joint>
 <!--/////////////////  LINK 4  //////////////////////// -->
+    <link name="link4">
+        <visual>
+            <origin xyz="0 0 0" rpy="0 0 0" />
+            <geometry>
+                <mesh filename="package://um_description/meshes/link4.STL" scale="1 1 1" />
+            </geometry>
+            <material name="Gray" />
+        </visual>
+    </link>
+    <joint name="joint5" type="revolute">
+        <parent link="link4" />
+        <child link="link5" />
+        <origin xyz="${JOINT5_COOR}" rpy="0 0 0" />
+        <axis xyz="0 1 0" />
+        <limit effort="${JOINT5_EFFORT}" lower="${JOINT5_LOWER}" upper="${JOINT5_UPPER}" velocity="${JOINT5_VEL}" />
+        <dynamics damping="${DAMPING}" friction="${FRICTION}" />
+    </joint>
 <!--/////////////////  LINK 5  //////////////////////// -->
+    <link name="link5">
+        <visual>
+            <origin xyz="0 0 0" rpy="0 0 0" />
+            <geometry>
+                <mesh filename="package://um_description/meshes/link5.STL" scale="1 1 1" />
+            </geometry>
+            <material name="Orange" />
+        </visual>
+    </link>
 </robot>

Commit message: add pkg um_moveit_config

File: um_description/urdf/um.urdf.xacro (robot description, xacro)
@@ -27,5 +27,7 @@
         <inertial>
             <mass value="${mass}" />
-            <inertia ixx="1.0" ixy="0" ixz="0" iyy="0.5" iyz="0" izz="1.0" />
+            <inertia ixx="0.001" ixy="0"    ixz="0"
+                                     iyy="0.001" iyz="0"
+                                                 izz="0.001" />
         </inertial>
     </xacro:macro>
@@ -35,4 +37,5 @@
     <xacro:property name="FRICTION" value="1" />
     <!-- Joint1 properties -->
+    <xacro:property name="JOINT1_COOR" value="0 0 0.5" />
     <xacro:property name="JOINT1_EFFORT" value="300" />
     <xacro:property name="JOINT1_LOWER" value="0" />
@@ -63,8 +66,14 @@
     <xacro:property name="JOINT5_UPPER" value="${M_PI/2}" />
     <xacro:property name="JOINT5_VEL" value="1.0" />
+ <!-- ///////////// WORLD LINK FOR GAZEBO ///////////// -->
+    <link name="world"/>
+    <joint name="fixed" type="fixed">
+        <parent link="world"/>
+        <child link="base_link"/>
+    </joint>
 <!-- ////////////////  BASE LINK  ///////////////////// -->
     <link name="base_link">
         <visual>
-            <origin xyz="0 0 0" rpy="0 0 0" />
+            <origin xyz="${JOINT1_COOR}" rpy="${M_PI} 0 0" />
             <geometry>
                 <mesh filename="package://um_description/meshes/base.STL" scale="1 1 1" />
@@ -73,5 +82,5 @@
         </visual>
         <collision>
-            <origin xyz="0 0 0" rpy="0 0 0" />
+            <origin xyz="${JOINT1_COOR}" rpy="${M_PI} 0 0" />
             <geometry>
                 <mesh filename="package://um_description/meshes/base.STL" scale="1 1 1" />
@@ -83,5 +92,5 @@
         <parent link="base_link"/>
         <child link="link1"/>
-        <origin xyz="0 0 0" rpy="0 0 0" />
+        <origin xyz="${JOINT1_COOR}" rpy="${M_PI} 0 0" />
         <axis xyz="1 0 0"/>
         <limit effort="${JOINT1_EFFORT}" lower="${JOINT1_LOWER}" upper="${JOINT1_UPPER}" velocity="${JOINT1_VEL}" />
@@ -247,4 +256,6 @@
         <plugin name="gazebo_ros_control" filename="libgazebo_ros_control.so">
             <robotNamespace>/um</robotNamespace>
+            <robotSimType>gazebo_ros_control/DefaultRobotHWSim</robotSimType>
+            <legacyModeNS>true</legacyModeNS>
         </plugin>
     </gazebo>
